Commit message: Update hande attachement

File: hande.urdf (robot description, URDF)
Before this commit: robot robotiq_hande, 6 links, 5 joints
Links:
- link robotiq_hande_coupler: geometry collision cylinder length=0.0169 radius=0.0385; visual mesh filename=package://robotiq_hande_description/meshes/io_coupler.dae
- link robotiq_hande_left_finger: geometry collision mesh filename=package://robotiq_hande_description/meshes/finger_collision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 scale=1.0 1.0 1.0; visual mesh filename=package://robotiq_hande_description/meshes/finger.dae scale=1.0 1.0 1.0
- link robotiq_hande_link: geometry collision cylinder length=0.10690000000000001 radius=0.0385; visual mesh filename=package://robotiq_hande_description/meshes/hande.dae scale=1.0 1.0 1.0
- link robotiq_hande_right_finger: geometry collision mesh filename=package://robotiq_hande_description/meshes/finger_collision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 scale=1.0 1.0 1.0; visual mesh filename=package://robotiq_hande_description/meshes/finger.dae scale=1.0 1.0 1.0
Joints:
- joint robotiq_hande_coupler_joint: parent tool0 -> hande_base

File: standalone_hande.urdf.xacro (robot description, xacro)
@@ -2,10 +2,10 @@
 <robot name="robotiq_hande" xmlns:xacro="http://ros.org/wiki/xacro">
   <link name="hande_base" />
-  <xacro:include filename="robotiq_hande_description/urdf/robotiq_hande_gripper.xacro" />
+  <xacro:include filename="src/robotiq_hande_description/urdf/robotiq_hande_gripper.xacro" />
   <!-- <xacro:robotiq_hande_gripper name="robotiq_hande" prefix="" parent="hande_base" /> -->
     <xacro:robotiq_hande_gripper
-        name="robotiq_hande_gripper"
-        prefix=""
-        parent="tool0"
+      name="robotiq_hande_gripper"
+      prefix=""
+      parent="hande_base"
         grip_pos_min="0.0"
         grip_pos_max="0.025"
